File: src/Hardware/GatorBallFB/GatorBallFB.kicad_sch (KiCad schematic)
At the start: 3 parts, among them IC1 DWM3000, U1 ESP32-WROOM-32E

Commit message: updated PCB
Parts:
- added C2, C3, C4, C5, C6: C, symbol Device:C
- added D1: SP0503BAHT, Package_TO_SOT_SMD:SOT-143, symbol Power_Protection:SP0503BAHT
- added J1: USB_C_Receptacle_USB2.0_14P, symbol Connector:USB_C_Receptacle_USB2.0_14P
- added R1, R2: R, symbol Device:R
- added R3: 1k, symbol Device:R
- added R4: 22.1k, symbol Device:R
- added R5: 47.5k, symbol Device:R
- added R7, R8: 5.1k, symbol Device:R
- added SW1, SW2: SW_Push, symbol Switch:SW_Push
- added U2: CP2102N-Axx-xQFN24, Package_DFN_QFN:QFN-24-1EP_4x4mm_P0.5mm_EP2.6x2.6mm, symbol Interface_USB:CP2102N-Axx-xQFN24
Connections:
- net +3V3: now also U1.2 (VDD), C2.1, C3.1, C4.1, R1.1, R2.1, R3.1, U2.6 (VDD)
- net GND: now also U1.1 (GND), U1.15 (GND), U1.38 (GND), U1.39 (GND), C2.2, C3.2, C4.2, C5.2, C6.2, D1.1 (A), J1.A1 (GND), J1.A12 (GND), J1.B1 (GND), J1.B12 (GND), J1.S1 (SHIELD), R5.2, R7.2, R8.1, SW1.1, SW2.1, U2.2 (GND), U2.25 (GND)
- net FLASH: now reaches U1.25 (IO0)
- net FLASH: now also R2.2, SW2.2
- net RESET: now reaches U1.3 (EN)
- net RESET: now also R1.2, SW1.2
- net UART_RX: now reaches U1.34 (RXD0/IO3)
- net UART_RX: now also U2.20 (RXD)
- net UART_TX: now reaches U1.35 (TXD0/IO1)
- net UART_TX: now also U2.21 (TXD)
- new net: R3.2, U2.9 (~{RST})
- new net: J1.B5 (CC2), R8.2
- new net: J1.A4 (VBUS), J1.A9 (VBUS), J1.B4 (VBUS), J1.B9 (VBUS), R4.1
- new net: J1.A5 (CC1), R7.1
- new net +5V: C5.1, C6.1, U2.7 (VREGIN)
- new net D+: D1.4 (K), J1.A6 (D+), J1.B6 (D+), U2.3 (D+)
- new net D-: D1.3 (K), J1.A7 (D-), J1.B7 (D-), U2.4 (D-)
- new net VBUS: D1.2 (K), R4.2, R5.1, U2.8 (VBUS)
Other:
- note added: "Pull this one GND to program"
- note added: "Pull this pin high to enable"

Commit message: schematic 99% complete
Parts:
- added C10, C7, C8, C9: C, symbol Device:C
- added IC2: RT9080-33GJ5, RT9080-33GJ5:SOT94P280X100-5N, symbol RT9080-33GJ5:RT9080-33GJ5
- added J2: Conn_01x02, symbol Connector_Generic:Conn_01x02
- added R10, R11, R6, R9: R, symbol Device:R
- added U3: MCP73831-2-OT, Package_TO_SOT_SMD:SOT-23-5, symbol Battery_Management:MCP73831-2-OT
Connections:
- net +3V3: now also C10.1, IC2.5 (VOUT), R10.2
- net GND: now also C10.2, C7.1, C8.2, C9.2, IC2.2 (GND), J2.2 (Pin_2), R11.1, R6.2, U3.2 (V_{SS})
- net VBUS: now also C7.2, U3.4 (V_{DD})
- new net: R6.1, U3.5 (PROG)
- new net: IC2.3 (EN), R9.2
- new net: IC2.4 (SNS), R10.1, R11.2
- new net VBAT: C8.1, C9.1, IC2.1 (VIN), J2.1 (Pin_1), R9.1, U3.3 (V_{BAT})

Commit message: fully routed pcb
Parts:
- removed C5, C6: C, symbol Device:C
- removed R10, R11: R, symbol Device:R
- added D2: D, LED_SMD:LED_0603_1608Metric, symbol Device:D
- added R12: 470, Resistor_SMD:R_0402_1005Metric, symbol Device:R
- C1, C2: value C -> 0.1u; footprint (none) -> Capacitor_SMD:C_0201_0603Metric
- C10: value C -> 1u; footprint (none) -> Capacitor_SMD:C_0201_0603Metric
- C3: value C -> 4.7uF; footprint (none) -> Capacitor_SMD:C_0201_0603Metric
- C4: value C -> 0.1uF; footprint (none) -> Capacitor_SMD:C_0201_0603Metric
- C7, C8: value C -> 4.7u; footprint (none) -> Capacitor_SMD:C_0201_0603Metric
- C9: value C -> 1uF; footprint (none) -> Capacitor_SMD:C_0201_0603Metric
- IC1: footprint DWM3000 -> DWM3000TR13:XCVR_DWM3000TR13
- IC2: footprint RT9080-33GJ5:SOT94P280X100-5N -> RT9080-33GJ5 (1):SOT94P280X100-5N
- J1: footprint (none) -> Connector_USB:USB_C_Receptacle_GCT_USB4085
- J2: footprint (none) -> Connector_JST:JST_PH_B2B-PH-SM4-TB_1x02-1MP_P2.00mm_Vertical
- R1, R2: value R -> 470; footprint (none) -> Resistor_SMD:R_0402_1005Metric
- R3, R4, R5, R7, R8: footprint (none) -> Resistor_SMD:R_0402_1005Metric
- R6: value R -> 2k; footprint (none) -> Resistor_SMD:R_0402_1005Metric
- R9: value R -> 10k; footprint (none) -> Resistor_SMD:R_0402_1005Metric
- SW1, SW2: footprint (none) -> Button_Switch_SMD:SW_SPST_EVPBF
Connections:
- net +5V is gone; now on net +3V3: U2.7 (VREGIN)
- net VBUS: now also D2.2 (A)
- net at U3.1 (STAT): now also R12.2
- new net: D2.1 (K), R12.1
Other:
- moved on the sheet: C7
